File: 01_bacca40/bacca40.sch (KiCad schematic (older format))
At the start: 145 parts, among them J1 TYPE-C-31-M12_13, J2 AVR-ISP-6_mod, K1 KEYSW, K10 KEYSW, K11 KEYSW, K12 KEYSW, K13 KEYSW, K14 KEYSW, K15 KEYSW, K16 KEYSW, K17 KEYSW, K18 KEYSW, K19 KEYSW, K2 KEYSW, K20 KEYSW, K21 KEYSW, K22 KEYSW, K23 KEYSW, K24 KEYSW, K25 KEYSW, K26 KEYSW, K27 KEYSW, K28 KEYSW, K29 KEYSW, K3 KEYSW, K30 KEYSW, K31 KEYSW, K32 KEYSW, K33 KEYSW, K34 KEYSW, K35 KEYSW, K36 KEYSW, K37 KEYSW, K38 KEYSW, K39 KEYSW, K4 KEYSW, K40 KEYSW, K41 KEYSW, K42 KEYSW, K43 KEYSW, K44 KEYSW, K45 KEYSW, K46 KEYSW, K47 KEYSW, K48 KEYSW, K49 KEYSW, K5 KEYSW, K50 KEYSW, K51 KEYSW, K52 KEYSW, K6 KEYSW, K7 KEYSW, K8 KEYSW, K9 KEYSW, SW1 SW_PUSH, SW2 Rotary_Encoder_Switch, U1 ATMEGA32U4, U3 USBLC6-2SC6, Y1 16MHz

Commit message: USB/MCU routed
Parts:
- removed D38, D40, D41, D42, D44, D45, D47, D50, D51, D52: D, Keeb_footprints:D_SOD-123_modified, symbol Ori-rescue:D-keyboard_parts
- removed H10, H11, H12, H13, H14, H15, H16, H17, H18, H8: MountingHole, random-keyboard-parts:plate_hole_4mm_tht, symbol Mechanical:MountingHole
- removed H19, H20, H21, H22: MountingHole, Keeb_footprints:MouseBite_IPC7351, symbol Mechanical:MountingHole
- removed K38, K40, K41, K42, K44, K45, K47, K50, K51, K52: KEYSW, Keeb_footprints:MX100, symbol Ori-rescue:KEYSW-keyboard_parts
- removed SW2: Rotary_Encoder_Switch, Keebio-Parts:RotaryEncoder_EC11, symbol Device:Rotary_Encoder_Switch
- D1, D10, D11, D12, D2, D3, D39, D4, D5, D6, D7, D8, D9: symbol Ori-rescue:D-keyboard_parts -> bacca40-rescue:D-keyboard_parts-Ori-rescue
- D13: renamed from D49; symbol Ori-rescue:D-keyboard_parts -> bacca40-rescue:D-keyboard_parts-Ori-rescue
- D14: renamed from D13; symbol Ori-rescue:D-keyboard_parts -> bacca40-rescue:D-keyboard_parts-Ori-rescue
- D15: renamed from D14; symbol Ori-rescue:D-keyboard_parts -> bacca40-rescue:D-keyboard_parts-Ori-rescue
- D16: renamed from D15; symbol Ori-rescue:D-keyboard_parts -> bacca40-rescue:D-keyboard_parts-Ori-rescue
- D17: renamed from D16; symbol Ori-rescue:D-keyboard_parts -> bacca40-rescue:D-keyboard_parts-Ori-rescue
- D18: renamed from D17; symbol Ori-rescue:D-keyboard_parts -> bacca40-rescue:D-keyboard_parts-Ori-rescue
- D19: renamed from D18; symbol Ori-rescue:D-keyboard_parts -> bacca40-rescue:D-keyboard_parts-Ori-rescue
- D20: renamed from D19; symbol Ori-rescue:D-keyboard_parts -> bacca40-rescue:D-keyboard_parts-Ori-rescue
- D21: renamed from D20; symbol Ori-rescue:D-keyboard_parts -> bacca40-rescue:D-keyboard_parts-Ori-rescue
- D22: renamed from D21; symbol Ori-rescue:D-keyboard_parts -> bacca40-rescue:D-keyboard_parts-Ori-rescue
- D23: renamed from D22; symbol Ori-rescue:D-keyboard_parts -> bacca40-rescue:D-keyboard_parts-Ori-rescue
- D24: renamed from D23; symbol Ori-rescue:D-keyboard_parts -> bacca40-rescue:D-keyboard_parts-Ori-rescue
- D25: renamed from D24; symbol Ori-rescue:D-keyboard_parts -> bacca40-rescue:D-keyboard_parts-Ori-rescue
- D26: renamed from D25; symbol Ori-rescue:D-keyboard_parts -> bacca40-rescue:D-keyboard_parts-Ori-rescue
- D27: renamed from D26; symbol Ori-rescue:D-keyboard_parts -> bacca40-rescue:D-keyboard_parts-Ori-rescue
- D28: renamed from D27; symbol Ori-rescue:D-keyboard_parts -> bacca40-rescue:D-keyboard_parts-Ori-rescue
- D29: renamed from D28; symbol Ori-rescue:D-keyboard_parts -> bacca40-rescue:D-keyboard_parts-Ori-rescue
- D30: renamed from D29; symbol Ori-rescue:D-keyboard_parts -> bacca40-rescue:D-keyboard_parts-Ori-rescue
- D31: renamed from D30; symbol Ori-rescue:D-keyboard_parts -> bacca40-rescue:D-keyboard_parts-Ori-rescue
- D32: renamed from D31; symbol Ori-rescue:D-keyboard_parts -> bacca40-rescue:D-keyboard_parts-Ori-rescue
- D33: renamed from D32; symbol Ori-rescue:D-keyboard_parts -> bacca40-rescue:D-keyboard_parts-Ori-rescue
- D34: renamed from D33; symbol Ori-rescue:D-keyboard_parts -> bacca40-rescue:D-keyboard_parts-Ori-rescue
- D35: renamed from D34; symbol Ori-rescue:D-keyboard_parts -> bacca40-rescue:D-keyboard_parts-Ori-rescue
- D36: renamed from D35; symbol Ori-rescue:D-keyboard_parts -> bacca40-rescue:D-keyboard_parts-Ori-rescue
- D37: renamed from D36; symbol Ori-rescue:D-keyboard_parts -> bacca40-rescue:D-keyboard_parts-Ori-rescue
- D38: renamed from D37; symbol Ori-rescue:D-keyboard_parts -> bacca40-rescue:D-keyboard_parts-Ori-rescue
- D40: renamed from D43; symbol Ori-rescue:D-keyboard_parts -> bacca40-rescue:D-keyboard_parts-Ori-rescue
- D41: renamed from D46; symbol Ori-rescue:D-keyboard_parts -> bacca40-rescue:D-keyboard_parts-Ori-rescue
- D42: renamed from D48; symbol Ori-rescue:D-keyboard_parts -> bacca40-rescue:D-keyboard_parts-Ori-rescue
- J1: symbol Ori-rescue:TYPE-C-31-M12_13-acheronSymbols -> bacca40-rescue:TYPE-C-31-M12_13-acheronSymbols-Ori-rescue
- J2: symbol Ori-rescue:AVR-ISP-6_mod-Connector -> bacca40-rescue:AVR-ISP-6_mod-Connector-Ori-rescue
- K1, K10, K11, K12, K2, K3, K4, K5, K6, K7, K8, K9: footprint Keeb_footprints:MX100 -> Keebio-Parts:MX_PCB_100H; symbol Ori-rescue:KEYSW-keyboard_parts -> bacca40-rescue:KEYSW-keyboard_parts-Ori-rescue
- K13: renamed from K49; footprint Keeb_footprints:MX100 -> Keebio-Parts:MX_PCB_100H; symbol Ori-rescue:KEYSW-keyboard_parts -> bacca40-rescue:KEYSW-keyboard_parts-Ori-rescue
- K14: renamed from K13; footprint Keeb_footprints:MX100 -> Keebio-Parts:MX_PCB_125H; symbol Ori-rescue:KEYSW-keyboard_parts -> bacca40-rescue:KEYSW-keyboard_parts-Ori-rescue
- K15: renamed from K14; footprint Keeb_footprints:MX100 -> Keebio-Parts:MX_PCB_100H; symbol Ori-rescue:KEYSW-keyboard_parts -> bacca40-rescue:KEYSW-keyboard_parts-Ori-rescue
- K16: renamed from K15; footprint Keeb_footprints:MX100 -> Keebio-Parts:MX_PCB_100H; symbol Ori-rescue:KEYSW-keyboard_parts -> bacca40-rescue:KEYSW-keyboard_parts-Ori-rescue
- K17: renamed from K16; footprint Keeb_footprints:MX100 -> Keebio-Parts:MX_PCB_100H; symbol Ori-rescue:KEYSW-keyboard_parts -> bacca40-rescue:KEYSW-keyboard_parts-Ori-rescue
- K18: renamed from K17; footprint Keeb_footprints:MX100 -> Keebio-Parts:MX_PCB_100H; symbol Ori-rescue:KEYSW-keyboard_parts -> bacca40-rescue:KEYSW-keyboard_parts-Ori-rescue
- K19: renamed from K18; footprint Keeb_footprints:MX100 -> Keebio-Parts:MX_PCB_100H; symbol Ori-rescue:KEYSW-keyboard_parts -> bacca40-rescue:KEYSW-keyboard_parts-Ori-rescue
- K20: renamed from K19; footprint Keeb_footprints:MX100 -> Keebio-Parts:MX_PCB_100H; symbol Ori-rescue:KEYSW-keyboard_parts -> bacca40-rescue:KEYSW-keyboard_parts-Ori-rescue
- K21: renamed from K20; footprint Keeb_footprints:MX100 -> Keebio-Parts:MX_PCB_100H; symbol Ori-rescue:KEYSW-keyboard_parts -> bacca40-rescue:KEYSW-keyboard_parts-Ori-rescue
- K22: renamed from K21; footprint Keeb_footprints:MX100 -> Keebio-Parts:MX_PCB_100H; symbol Ori-rescue:KEYSW-keyboard_parts -> bacca40-rescue:KEYSW-keyboard_parts-Ori-rescue
- K23: renamed from K22; footprint Keeb_footprints:MX100 -> Keebio-Parts:MX_PCB_100H; symbol Ori-rescue:KEYSW-keyboard_parts -> bacca40-rescue:KEYSW-keyboard_parts-Ori-rescue
- K24: renamed from K23; footprint Keeb_footprints:MX100 -> Keebio-Parts:MX_PCB_100H; symbol Ori-rescue:KEYSW-keyboard_parts -> bacca40-rescue:KEYSW-keyboard_parts-Ori-rescue
- K25: renamed from K24; footprint Keeb_footprints:MX100 -> Keebio-Parts:MX_PCB_175H; symbol Ori-rescue:KEYSW-keyboard_parts -> bacca40-rescue:KEYSW-keyboard_parts-Ori-rescue
- K26: renamed from K25; footprint Keeb_footprints:MX100 -> Keebio-Parts:MX_PCB_175H; symbol Ori-rescue:KEYSW-keyboard_parts -> bacca40-rescue:KEYSW-keyboard_parts-Ori-rescue
- K27: renamed from K26; footprint Keeb_footprints:MX100 -> Keebio-Parts:MX_PCB_100H; symbol Ori-rescue:KEYSW-keyboard_parts -> bacca40-rescue:KEYSW-keyboard_parts-Ori-rescue
- K28: renamed from K27; footprint Keeb_footprints:MX100 -> Keebio-Parts:MX_PCB_100H; symbol Ori-rescue:KEYSW-keyboard_parts -> bacca40-rescue:KEYSW-keyboard_parts-Ori-rescue
- K29: renamed from K28; footprint Keeb_footprints:MX100 -> Keebio-Parts:MX_PCB_100H; symbol Ori-rescue:KEYSW-keyboard_parts -> bacca40-rescue:KEYSW-keyboard_parts-Ori-rescue
- K30: renamed from K29; footprint Keeb_footprints:MX100 -> Keebio-Parts:MX_PCB_100H; symbol Ori-rescue:KEYSW-keyboard_parts -> bacca40-rescue:KEYSW-keyboard_parts-Ori-rescue
- K31: renamed from K30; footprint Keeb_footprints:MX100 -> Keebio-Parts:MX_PCB_100H; symbol Ori-rescue:KEYSW-keyboard_parts -> bacca40-rescue:KEYSW-keyboard_parts-Ori-rescue
- K32: renamed from K31; footprint Keeb_footprints:MX100 -> Keebio-Parts:MX_PCB_100H; symbol Ori-rescue:KEYSW-keyboard_parts -> bacca40-rescue:KEYSW-keyboard_parts-Ori-rescue
- K33: renamed from K32; footprint Keeb_footprints:MX100 -> Keebio-Parts:MX_PCB_100H; symbol Ori-rescue:KEYSW-keyboard_parts -> bacca40-rescue:KEYSW-keyboard_parts-Ori-rescue
- K34: renamed from K33; footprint Keeb_footprints:MX100 -> Keebio-Parts:MX_PCB_100H; symbol Ori-rescue:KEYSW-keyboard_parts -> bacca40-rescue:KEYSW-keyboard_parts-Ori-rescue
- K35: renamed from K34; footprint Keeb_footprints:MX100 -> Keebio-Parts:MX_PCB_100H; symbol Ori-rescue:KEYSW-keyboard_parts -> bacca40-rescue:KEYSW-keyboard_parts-Ori-rescue
- K36: renamed from K35; footprint Keeb_footprints:MX100 -> Keebio-Parts:MX_PCB_125H; symbol Ori-rescue:KEYSW-keyboard_parts -> bacca40-rescue:KEYSW-keyboard_parts-Ori-rescue
- K37: renamed from K36; footprint Keeb_footprints:MX100 -> Keebio-Parts:MX_PCB_100H; symbol Ori-rescue:KEYSW-keyboard_parts -> bacca40-rescue:KEYSW-keyboard_parts-Ori-rescue
- K38: renamed from K37; footprint Keeb_footprints:MX100 -> Keebio-Parts:MX_PCB_125H; symbol Ori-rescue:KEYSW-keyboard_parts -> bacca40-rescue:KEYSW-keyboard_parts-Ori-rescue
- K39: footprint Keeb_footprints:MX100 -> Keebio-Parts:MX_PCB_125H; symbol Ori-rescue:KEYSW-keyboard_parts -> bacca40-rescue:KEYSW-keyboard_parts-Ori-rescue
- K40: renamed from K43; footprint Keeb_footprints:MX100 -> Keebio-Parts:MX_Plate_625H; symbol Ori-rescue:KEYSW-keyboard_parts -> bacca40-rescue:KEYSW-keyboard_parts-Ori-rescue
- K41: renamed from K46; footprint Keeb_footprints:MX100 -> Keebio-Parts:MX_PCB_125H; symbol Ori-rescue:KEYSW-keyboard_parts -> bacca40-rescue:KEYSW-keyboard_parts-Ori-rescue
- K42: renamed from K48; footprint Keeb_footprints:MX100 -> Keebio-Parts:MX_PCB_125H; symbol Ori-rescue:KEYSW-keyboard_parts -> bacca40-rescue:KEYSW-keyboard_parts-Ori-rescue
- LED1: symbol Ori-rescue:LED-keyboard_parts -> bacca40-rescue:LED-keyboard_parts-Ori-rescue
- SW1: symbol Ori-rescue:SW_PUSH-keyboard_parts -> bacca40-rescue:SW_PUSH-keyboard_parts-Ori-rescue
- U1: symbol Ori-rescue:ATMEGA32U4-keyboard_parts -> bacca40-rescue:ATMEGA32U4-keyboard_parts-Ori-rescue
- U3: symbol Ori-rescue:Power_Protection_USBLC6-2SC6-shark-cache -> bacca40-rescue:Power_Protection_USBLC6-2SC6-shark-cache-Ori-rescue
Connections:
- net col6: now also K40.1
- net col7: no longer K40.1
Other:
- note removed: "Breakaway Screw Holes"
- note removed: "Dori Screw Holes"
- note removed: "Mousebites"
- moved on the sheet: D13, D40, K13, K40

Commit message: Fully routed?
Parts:
- K40: footprint Keebio-Parts:MX_Plate_625H -> Keebio-Parts:MX_PCB_625H
Connections:
- net enc0a is gone; now on net col12: U1.21 (PD3/TXD1)
- net col0: now also K1.1, K14.1, K26.1, K38.1, U1.26 (T1/PD6); no longer K12.1, K25.1, K37.1, K42.1, U1.11 (PB3/MISO)
- net col1: now also K15.1, K2.1, K27.1, U1.31 (PC6); no longer K1.1, K14.1, K26.1, K38.1, U1.27 (T0/PD7)
- net col10: now also K11.1, K24.1, K36.1, U1.10 (PB2/MOSI); no longer K10.1, K23.1, K35.1, K41.1, U1.9 (PB1/SCK)
- net col11: now also K12.1, K25.1, K37.1, K42.1, U1.11 (PB3/MISO); no longer K11.1, K24.1, K36.1, U1.10 (PB2/MOSI)
- net col12: no longer U1.31 (PC6)
- net col2: now also K16.1, K28.1, K3.1, K39.1, U1.12 (PB7/~RTS); no longer K15.1, K2.1, K27.1, U1.22 (PD5/XCK1)
- net col3: now also K17.1, K29.1, K4.1, U1.38 (PF5); no longer K16.1, K28.1, K3.1, K39.1, U1.12 (PB7/~RTS)
- net col4: now also K18.1, K30.1, K5.1, U1.39 (PF4); no longer K17.1, K29.1, K4.1, U1.38 (PF5)
- net col5: now also K19.1, K31.1, K40.1, K6.1, U1.40 (PF1); no longer K18.1, K30.1, K5.1, U1.39 (PF4)
- net col6: now also K20.1, K32.1, K7.1, U1.41 (PF0); no longer K19.1, K31.1, K40.1, K6.1, U1.40 (PF1)
- net col7: now also K21.1, K33.1, K8.1, U1.1 (PE6/AIN0); no longer K20.1, K32.1, K7.1, U1.41 (PF0)
- net col8: now also K22.1, K34.1, K9.1, U1.8 (PB0/SS); no longer K21.1, K33.1, K8.1, U1.1 (PE6/AIN0)
- net col9: now also K10.1, K23.1, K35.1, K41.1, U1.9 (PB1/SCK); no longer K22.1, K34.1, K9.1, U1.8 (PB0/SS)
- net row2: now also U1.32 (PC7); no longer U1.25 (ICP1/PD4)
- net row3: now also U1.25 (ICP1/PD4); no longer U1.26 (T1/PD6)
- net enc0b: no longer names the net of U1.20 (PD2/RXD1)
- no-connect marks 9 -> 10
Changed lines of the file:
@@
 Text GLabel 2800 6600 2    50   BiDi ~ 0
 DBUS-
-Text GLabel 7450 6000 2    50   Output ~ 0
-row1
-Text GLabel 5300 7400 0    50   Output ~ 0
+Text GLabel 7450 6600 2    50   Output ~ 0
+col1
+Text GLabel 5300 6400 0    50   Output ~ 0
 col2
-Text GLabel 5300 6400 0    50   Output ~ 0
-col3
 Text GLabel 5300 6200 0    50   Output ~ 0
-col11
+col10
 Text GLabel 5300 6100 0    50   Output ~ 0
-col10
+col9
 Text GLabel 5300 6000 0    50   Output ~ 0
-col9
+col8
 Text GLabel 5300 5300 0    50   Output ~ 0
-col8
+col7
 Text GLabel 7450 6100 2    50   Output ~ 0
 row0
@@
 $EndComp
 Text GLabel 7450 5800 2    50   Output ~ 0
+col4
+Text GLabel 7450 5700 2    50   Output ~ 0
 col5
-Text GLabel 7450 5700 2    50   Output ~ 0
+Text GLabel 7450 5600 2    50   Output ~ 0
 col6
-Text GLabel 7450 5600 2    50   Output ~ 0
-col7
 NoConn ~ 7450 5500
 Text GLabel 5300 9300 2    50   BiDi ~ 0
@@
 	0    1    1    0
 $EndComp
-Text GLabel 7450 5900 2    50   Output ~ 0
-col4
-Text GLabel 7450 7100 2    50   Output ~ 0
+Text GLabel 7450 7200 2    50   Output ~ 0
 row3
-Text GLabel 7450 7200 2    50   Output ~ 0
+Text GLabel 7450 6500 2    50   Output ~ 0
 row2
 $Comp
@@
 ISP_Reset
 Text GLabel 13350 1700 1    50   Input ~ 0
-col0
+col11
 Text GLabel 5300 6300 0    50   Output ~ 0
-col0
+col11
 Wire Wire Line
 	4950 6500 4950 6650
@@
 F 0 "K40" H 7900 3900 60  0000 C CNN
 F 1 "KEYSW" H 7900 3800 60  0001 C CNN
-F 2 "Keebio-Parts:MX_Plate_625H" H 7900 3900 60  0001 C CNN
+F 2 "Keebio-Parts:MX_PCB_625H" H 7900 3900 60  0001 C CNN
 F 3 "" H 7900 3900 60  0000 C CNN
 	1    7900 3900
@@
 Connection ~ 11650 2500
 Text GLabel 4000 1700 1    50   Input ~ 0
+col0
+Text GLabel 4850 1700 1    50   Input ~ 0
 col1
-Text GLabel 4850 1700 1    50   Input ~ 0
+Text GLabel 5700 1700 1    50   Input ~ 0
 col2
-Text GLabel 5700 1700 1    50   Input ~ 0
+Text GLabel 6550 1700 1    50   Input ~ 0
 col3
-Text GLabel 6550 1700 1    50   Input ~ 0
+Text GLabel 7400 1700 1    50   Input ~ 0
 col4
-Text GLabel 7400 1700 1    50   Input ~ 0
+Text GLabel 8250 1700 1    50   Input ~ 0
 col5
-Text GLabel 8250 1700 1    50   Input ~ 0
+Text GLabel 9100 1700 1    50   Input ~ 0
 col6
-Text GLabel 9100 1700 1    50   Input ~ 0
+Text GLabel 9950 1700 1    50   Input ~ 0
 col7
-Text GLabel 9950 1700 1    50   Input ~ 0
+Text GLabel 10800 1700 1    50   Input ~ 0
 col8
-Text GLabel 10800 1700 1    50   Input ~ 0
+Text GLabel 11650 1700 1    50   Input ~ 0
 col9
-Text GLabel 11650 1700 1    50   Input ~ 0
+Text GLabel 12500 1700 1    50   Input ~ 0
 col10
-Text GLabel 12500 1700 1    50   Input ~ 0
-col11
-Text GLabel 5300 7200 0    50   Output ~ 0
-enc0b
-Text GLabel 5300 7300 0    50   Output ~ 0
-enc0a
-Text GLabel 7450 7000 2    50   Output ~ 0
-col1
+Text GLabel 7450 7100 2    50   Output ~ 0
+col0
 Text GLabel 2800 4250 0    50   Input ~ 0
 row3
@@
 Text GLabel 6850 9050 3    50   Input ~ 0
 ISP_Reset
-Text GLabel 7450 6600 2    50   Output ~ 0
+Text GLabel 5300 7300 0    50   Output ~ 0
 col12
-NoConn ~ 7450 6500
+NoConn ~ 7450 7000
 NoConn ~ 7450 6700
 NoConn ~ 7450 6800
 NoConn ~ 7450 6900
-NoConn ~ 5300 7100
+NoConn ~ 5300 7200
 NoConn ~ 5300 7000
 Connection ~ 3300 2150
@@
 Wire Wire Line
 	7550 4250 10950 4250
+NoConn ~ 5300 7100
+Text GLabel 7450 5900 2    50   Output ~ 0
+col3
+Text GLabel 7450 6000 2    50   Output ~ 0
+row1
 $EndSCHEMATC
